File: wfipic32host.brd (EAGLE design)
At the start: 95.2 x 43.6 mm, 78 parts, among them IC1 BMA490L, IC2 TCAN330GD, IC3 WFI32E01PE-I, J1 MLE-105-01-G-DV, J2 MLE-105-01-G-DV, J3 MLE-105-01-G-DV, J4 MLE-105-01-G-DV, U1 PIC32MK0512MCJ048T-I/Y8XTQFP4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, U2 MAX6126B30

Commit message: up
Parts:
- added SJ3: sdo1_jmp, jumper:SJ_2
- moved GND_POINTS 1.27 mm to (26.7, 24.1)
- moved L1 1.27 mm to (14.0, 29.2)
Connections:
- removed net WFI_C9_SIG: IC3.18, SV4.3
- new net DIS_SDO: SJ3.2, SV2.2
- new net WFI_SDO1: IC3.18, SJ3.1, SV4.3
- net SDO1: now also SJ3.3; no longer IC3.23, SV2.2
Routing:
- net WFI_SDO1: track 0.00 -> 67.3 mm, vias 0 -> 3
- net WFI_C9_SIG: track 33.2 -> 0.00 mm, vias 1 -> 0
- net SDO1: track 122.1 -> 112.8 mm, vias 6 -> 7
- net DIS_SDO: track 0.00 -> 7.40 mm, vias 0 -> 1
- net AVDD: track 44.2 -> 42.9 mm
- net VSS: track 224.4 -> 223.7 mm
Other:
- board text added: "PIC32MK-CANFD HOST V1.9"
- board text removed: "PIC32MK-CANFD HOST V1.8"
