File: wfipic32host.sch (EAGLE design)
At the start: 67 parts, among them IC1 BMA490L, IC2 TCAN330GD, IC3 WFI32E01PE-I, J1 MLE-105-01-G-DV, J2 MLE-105-01-G-DV, J3 MLE-105-01-G-DV, J4 MLE-105-01-G-DV, U1 PIC32MK0512MCJ048T-I/Y8XTQFP4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, U2 MAX6126B30

Commit message: up
Connections:
- net VSS: now also IC3.EP_1, IC3.EP_2, IC3.EP_3
Changed lines of the file:
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@@
 </segment>
 </net>
-<net name="VSS" class="2">
+<net name="VSS" class="1">
 <segment>
 <wire x1="7.62" y1="124.46" x2="10.16" y2="124.46" width="0.1524" layer="91"/>
@@
 <junction x="254" y="17.78"/>
 </segment>
+<segment>
+<wire x1="398.78" y1="7.62" x2="401.32" y2="7.62" width="0.1524" layer="91"/>
+<pinref part="IC3" gate="G$1" pin="EP_1"/>
+<junction x="401.32" y="7.62"/>
+<wire x1="401.32" y1="7.62" x2="411.48" y2="7.62" width="0.1524" layer="91"/>
+<junction x="411.48" y="7.62"/>
+<junction x="398.78" y="7.62"/>
+<label x="414.02" y="7.62" size="1.778" layer="95"/>
+</segment>
+<segment>
+<wire x1="398.78" y1="5.08" x2="411.48" y2="5.08" width="0.1524" layer="91"/>
+<pinref part="IC3" gate="G$1" pin="EP_2"/>
+<junction x="398.78" y="5.08"/>
+<junction x="411.48" y="5.08"/>
+<label x="414.02" y="5.08" size="1.778" layer="95"/>
+</segment>
+<segment>
+<wire x1="398.78" y1="2.54" x2="411.48" y2="2.54" width="0.1524" layer="91"/>
+<pinref part="IC3" gate="G$1" pin="EP_3"/>
+<junction x="398.78" y="2.54"/>
+<junction x="411.48" y="2.54"/>
+<label x="414.02" y="2.54" size="1.778" layer="95"/>
+</segment>
 </net>
