File: wfipic32host.sch (EAGLE design)
At the start: 67 parts, among them IC1 BMA490L, IC2 TCAN330GD, IC3 WFI32E01PE-I, J1 MLE-105-01-G-DV, J2 MLE-105-01-G-DV, J3 MLE-105-01-G-DV, J4 MLE-105-01-G-DV, U1 PIC32MK0512MCJ048T-I/Y8XTQFP4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, U2 MAX6126B30

Commit message: up
Parts:
- added C24: 0.1uf, rcl:C-USC0805
- added C25: 10uf, rcl:C-USC0805
- added JP3: USB_HEADER, pinhead:PINHD-1X6
Connections:
- net N$6 renamed TP2_SIG
- removed net N$10: IC2.TXD, S1.6
- removed net N$11: IC2.RXD, S1.3
- removed net N$5: TP1.TP, U1.AN11/CVD11/C1IN2-/FLT4/RC11
- new net AN2_WFI: IC3.AN2_/_CVD2_/_CVDR2_/_CVDT5_/_USBID_/_RPB2, JP3.4, SV5.1
- new net C1RX_SIG: IC2.RXD, IC3.TMS_/_AN6_/_CVD6_/_CVDR6_/_RPB6, S1.3
- new net C1TX_SIG: IC2.TXD, IC3.ANA0_/_RPB12, S1.6
- new net D_NEG: IC3.USB_D-, JP3.2
- new net D_POS: IC3.USB_D+, JP3.3
- new net IMU_INT2_SIG: IC3.AN14_/_ANN0_/_CVD14_/_CVDR14_/_RPA14, SV5.2
- new net OSC_OUT: IC3.SOSCO/PK15, J4.4
- new net TP1_SIG: IC3.AN15_/_ANN1_/_CVD15_/_CVDR15_/_RPA13, TP1.TP, U1.AN11/CVD11/C1IN2-/FLT4/RC11
- new net VBUS: IC3.VBUS, JP3.1
- new net VBUSON: IC3.AN1_/_CVD1_/_CVDR1_/_CVDT6_/_VBUSON_/_RPB1, JP3.6
- new net WFI_C15_SIG: IC3.CVDT13_/_ETXD0_/_RPC15, SV4.2
- new net WFI_C9_SIG: IC3.CVDT7_/_ERXERR_/_RPC9, SV4.3
- net AN1: now also IC3.TDI_/_PGD4_/_AN9_/_CVD9_/_CVDR9_/_RPB9
- net BMA_INT2: now also IC3.PTA_BT_PRIO_/_RPK6
- net DAC1: now also IC3.SDA1_/_RPA5
- net DIS_CS: now also IC3.!SPI1CS_!/_RPA1
- net DIS_MODE: now also IC3.CVDT8_/_ERXD1_/_RPC10
- net DIS_RESET: now also IC3.CVDT10_/_ETH_CLK_OUT_/_RPC12
- net EXT_SW2: now also IC3.AN17_/_CVD17_/_CVDR17_/_INT0_/_RPA10
- net GREEN_LED: now also IC3.RF_FE_2_/_RPK3
- net IMU_CS: now also IC3.TDO_/_AN7_/_CVD7_/_CVDR7_/_RPB7
- net INDX2: now also IC3.SCL1_/_RPA4
- net OSC_MCU: now also IC3.SOSCI/PB15
- net PGC_C1RX: now also IC3.PGC2_/_AN4_/_CVD4_/_CVDR4_/_CVDT3_/_RPB4
- net PGD_C1TX: now also IC3.PGD2_/_AN5_/_CVD5_/_CVDR5_/_CVDT2_/_RTCC_/_RPB5
- net PWM1H: now also IC3.CVDT14_/_ERXDV_/_RPK12
- net PWM1L: now also IC3.CVDT9_/_ERXD0_/_RPC11
- net QEA2: now also IC3.CVDT16_/_EMDC_/_RPK14
- net QEB2: now also IC3.CVDT15_/_EMDIO_/_RPK13
- net RED_LED: now also IC3.RF_FE_4_/_RPK1
- net SCK1: now also IC3.SCK1_/_RPC6
- net SCK2: now also IC3.SCK2_/_RPA11
- net SDI1: now also IC3.SDI1_/_RPC7
- net SDI2: now also IC3.PTA_WLAN_ACTIVE_/_RPK5
- net SDO1: now also IC3.SDO1_/_RPC8
- net SDO2: now also IC3.BT_CLK_OUT_/_RPK4
- net U1RX: now also IC3.CVDT11_/_ETXEN_/_RPC13
- net U1TX: now also IC3.CVDT12_/_ETXD1_/_RPC14
- net VDD: now also C24.1, C25.1
- net VREF+: now also IC3.TCK_/_PGC4_/_AN8_/_CVD8_/_CVDR8_/_RPB8
- net VSS: now also C24.2, C25.2, IC3.EP_1, IC3.EP_2, IC3.EP_3, JP3.5; no longer SV4.2, SV4.3, SV5.1, SV5.2
Other:
- moved on the sheet: SV4

Commit message: up
Connections:
- net U1RX renamed U1RX_U3RX
- net U1TX renamed U1TX_U3TX
- removed net AN0: J2.3, U1.OA2OUT/AN0/C2IN4-/C4IN3-/RPA0/RA0
- removed net C1RX_SIG: IC2.RXD, IC3.TMS_/_AN6_/_CVD6_/_CVDR6_/_RPB6, S1.3
- removed net C1TX_SIG: IC2.TXD, IC3.ANA0_/_RPB12, S1.6
- removed net DAC1: IC3.SDA1_/_RPA5, J2.9, U1.DAC1/AN48/CVD48/RPC10/RC10
- new net AN0_AN6: IC3.TMS_/_AN6_/_CVD6_/_CVDR6_/_RPB6, J2.3, U1.OA2OUT/AN0/C2IN4-/C4IN3-/RPA0/RA0
- new net C1RX_SIG_C2RX: IC2.RXD, IC3.PTA_BT_ACTIVE_/_RPK7, S1.3
- new net C1TX_SIG_C2TX: IC2.TXD, IC3.SDA1_/_RPA5, S1.6
- new net DAC1_RB12: IC3.ANA0_/_RPB12, J2.9, U1.DAC1/AN48/CVD48/RPC10/RC10
Changed lines of the file:
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@@
 </segment>
 </net>
-<net name="U1RX" class="0">
+<net name="U1RX_U3RX" class="0">
 <segment>
 <pinref part="U1" gate="A" pin="OA3IN-/AN7/CVD7/C3IN1-/C4IN1-/RPC1/RC1"/>
@@
 </segment>
 </net>
-<net name="U1TX" class="0">
+<net name="U1TX_U3TX" class="0">
 <segment>
 <wire x1="170.18" y1="121.92" x2="157.48" y2="121.92" width="0.1524" layer="91"/>
@@
 </segment>
 </net>
-<net name="AN0" class="0">
+<net name="AN0_AN6" class="0">
 <segment>
 <pinref part="U1" gate="A" pin="OA2OUT/AN0/C2IN4-/C4IN3-/RPA0/RA0"/>
@@
 <wire x1="170.18" y1="86.36" x2="157.48" y2="86.36" width="0.1524" layer="91"/>
 <pinref part="J2" gate="G$1" pin="3"/>
-<label x="147.32" y="86.36" size="1.778" layer="95"/>
+<label x="144.78" y="86.36" size="1.778" layer="95"/>
 <junction x="170.18" y="86.36"/>
 <junction x="157.48" y="86.36"/>
+</segment>
+<segment>
+<wire x1="411.48" y1="30.48" x2="398.78" y2="30.48" width="0.1524" layer="91"/>
+<pinref part="IC3" gate="G$1" pin="TMS_/_AN6_/_CVD6_/_CVDR6_/_RPB6"/>
+<junction x="398.78" y="30.48"/>
+<junction x="411.48" y="30.48"/>
+<label x="414.02" y="30.48" size="1.778" layer="95"/>
 </segment>
 </net>
@@
 </segment>
 </net>
-<net name="DAC1" class="0">
+<net name="DAC1_RB12" class="0">
 <segment>
 <pinref part="U1" gate="A" pin="DAC1/AN48/CVD48/RPC10/RC10"/>
@@
 </segment>
 <segment>
-<wire x1="398.78" y1="63.5" x2="411.48" y2="63.5" width="0.1524" layer="91"/>
-<pinref part="IC3" gate="G$1" pin="SDA1_/_RPA5"/>
-<junction x="398.78" y="63.5"/>
-<junction x="411.48" y="63.5"/>
-<label x="414.02" y="63.5" size="1.778" layer="95"/>
+<wire x1="398.78" y1="33.02" x2="411.48" y2="33.02" width="0.1524" layer="91"/>
+<pinref part="IC3" gate="G$1" pin="ANA0_/_RPB12"/>
+<junction x="398.78" y="33.02"/>
+<junction x="411.48" y="33.02"/>
+<label x="416.56" y="33.02" size="1.778" layer="95"/>
 </segment>
 </net>
@@
 </segment>
 </net>
-<net name="C1TX_SIG" class="0">
+<net name="C1TX_SIG_C2TX" class="0">
 <segment>
 <pinref part="IC2" gate="G$1" pin="TXD"/>
@@
 </segment>
 <segment>
-<wire x1="424.18" y1="33.02" x2="398.78" y2="33.02" width="0.1524" layer="91"/>
-<pinref part="IC3" gate="G$1" pin="ANA0_/_RPB12"/>
-<junction x="398.78" y="33.02"/>
-<junction x="424.18" y="33.02"/>
-<label x="414.02" y="33.02" size="1.778" layer="95"/>
-</segment>
-</net>
-<net name="C1RX_SIG" class="0">
+<wire x1="424.18" y1="63.5" x2="398.78" y2="63.5" width="0.1524" layer="91"/>
+<pinref part="IC3" gate="G$1" pin="SDA1_/_RPA5"/>
+<junction x="398.78" y="63.5"/>
+<junction x="424.18" y="63.5"/>
+<label x="416.56" y="63.5" size="1.778" layer="95"/>
+</segment>
+</net>
+<net name="C1RX_SIG_C2RX" class="0">
 <segment>
 <pinref part="IC2" gate="G$1" pin="RXD"/>
@@
 </segment>
 <segment>
-<wire x1="424.18" y1="30.48" x2="398.78" y2="30.48" width="0.1524" layer="91"/>
-<pinref part="IC3" gate="G$1" pin="TMS_/_AN6_/_CVD6_/_CVDR6_/_RPB6"/>
-<junction x="398.78" y="30.48"/>
-<junction x="424.18" y="30.48"/>
-<label x="414.02" y="30.48" size="1.778" layer="95"/>
+<wire x1="266.7" y1="2.54" x2="241.3" y2="2.54" width="0.1524" layer="91"/>
+<pinref part="IC3" gate="G$1" pin="PTA_BT_ACTIVE_/_RPK7"/>
+<junction x="266.7" y="2.54"/>
+<junction x="241.3" y="2.54"/>
+<label x="236.22" y="2.54" size="1.778" layer="95"/>
 </segment>
 </net>
@@
 <junction x="266.7" y="60.96"/>
 <junction x="256.54" y="60.96"/>
+<label x="238.76" y="60.96" size="1.778" layer="95"/>
 </segment>
 <segment>
@@
 <junction x="266.7" y="58.42"/>
 <junction x="256.54" y="58.42"/>
-</segment>
-<segment>
+<label x="238.76" y="58.42" size="1.778" layer="95"/>
+</segment>
+<segment>

Commit message: up
Connections:
- net AN1 renamed AN1_AN9
Changed lines of the file:
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@@
 </segment>
 </net>
-<net name="AN1" class="0">
+<net name="AN1_AN9" class="0">
 <segment>
 <pinref part="U1" gate="A" pin="OA2IN+/AN1/C2IN1+/RPA1/RA1"/>

Commit message: up
Parts:
- added C26, C27, C28, C29, C30, C31, C32: 10pf, rcl:C-USC0402
Connections:
- net BMA_INT2: now also C29.1
- net C1RX_SIG_C2RX: now also C26.1
- net MCLR_SIG: now also C28.1
- net SDI2: now also C27.1
- net SDO1: now also C31.1
- net SDO2: now also C30.1
- net VDD: now also C32.1
- net VSS: now also C26.2, C27.2, C28.2, C29.2, C30.2, C31.2, C32.2
Changed lines of the file:
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@@
 <part name="VSS26" library="supply1" library_urn="urn:adsk.eagle:library:371" deviceset="VSS" device=""/>
 <part name="VSS46" library="supply1" library_urn="urn:adsk.eagle:library:371" deviceset="VSS" device=""/>
+<part name="C26" library="rcl" library_urn="urn:adsk.eagle:library:334" deviceset="C-US" device="C0402" package3d_urn="urn:adsk.eagle:package:23626/2" value="10pf"/>
+<part name="VSS47" library="supply1" library_urn="urn:adsk.eagle:library:371" deviceset="VSS" device=""/>
+<part name="C27" library="rcl" library_urn="urn:adsk.eagle:library:334" deviceset="C-US" device="C0402" package3d_urn="urn:adsk.eagle:package:23626/2" value="10pf"/>
+<part name="C28" library="rcl" library_urn="urn:adsk.eagle:library:334" deviceset="C-US" device="C0402" package3d_urn="urn:adsk.eagle:package:23626/2" value="10pf"/>
+<part name="C29" library="rcl" library_urn="urn:adsk.eagle:library:334" deviceset="C-US" device="C0402" package3d_urn="urn:adsk.eagle:package:23626/2" value="10pf"/>
+<part name="C30" library="rcl" library_urn="urn:adsk.eagle:library:334" deviceset="C-US" device="C0402" package3d_urn="urn:adsk.eagle:package:23626/2" value="10pf"/>
+<part name="C31" library="rcl" library_urn="urn:adsk.eagle:library:334" deviceset="C-US" device="C0402" package3d_urn="urn:adsk.eagle:package:23626/2" value="10pf"/>
+<part name="C32" library="rcl" library_urn="urn:adsk.eagle:library:334" deviceset="C-US" device="C0402" package3d_urn="urn:adsk.eagle:package:23626/2" value="10pf"/>
 </parts>
 <sheets>
@@
 <instance part="VSS46" gate="G$1" x="398.78" y="-7.62" smashed="yes">
 <attribute name="VALUE" x="396.24" y="-12.7" size="1.778" layer="96" rot="R90"/>
+</instance>
+<instance part="C26" gate="G$1" x="279.4" y="-30.48" smashed="yes">
+<attribute name="NAME" x="280.416" y="-29.845" size="1.778" layer="95"/>
+<attribute name="VALUE" x="280.416" y="-34.671" size="1.778" layer="96"/>
+</instance>
+<instance part="VSS47" gate="G$1" x="325.12" y="-38.1" smashed="yes">
+<attribute name="VALUE" x="322.58" y="-43.18" size="1.778" layer="96" rot="R90"/>
+</instance>
+<instance part="C27" gate="G$1" x="292.1" y="-30.48" smashed="yes">
+<attribute name="NAME" x="293.116" y="-29.845" size="1.778" layer="95"/>
+<attribute name="VALUE" x="293.116" y="-34.671" size="1.778" layer="96"/>
+</instance>
+<instance part="C28" gate="G$1" x="304.8" y="-30.48" smashed="yes">
+<attribute name="NAME" x="305.816" y="-29.845" size="1.778" layer="95"/>
+<attribute name="VALUE" x="305.816" y="-34.671" size="1.778" layer="96"/>
+</instance>
+<instance part="C29" gate="G$1" x="320.04" y="-30.48" smashed="yes">
+<attribute name="NAME" x="321.056" y="-29.845" size="1.778" layer="95"/>
+<attribute name="VALUE" x="321.056" y="-34.671" size="1.778" layer="96"/>
+</instance>
+<instance part="C30" gate="G$1" x="332.74" y="-30.48" smashed="yes">
+<attribute name="NAME" x="333.756" y="-29.845" size="1.778" layer="95"/>
+<attribute name="VALUE" x="333.756" y="-34.671" size="1.778" layer="96"/>
+</instance>
+<instance part="C31" gate="G$1" x="342.9" y="-30.48" smashed="yes">
+<attribute name="NAME" x="343.916" y="-29.845" size="1.778" layer="95"/>
+<attribute name="VALUE" x="343.916" y="-34.671" size="1.778" layer="96"/>
+</instance>
+<instance part="C32" gate="G$1" x="353.06" y="-30.48" smashed="yes">
+<attribute name="NAME" x="354.076" y="-29.845" size="1.778" layer="95"/>
+<attribute name="VALUE" x="354.076" y="-34.671" size="1.778" layer="96"/>
 </instance>
 </instances>
@@
 <label x="414.02" y="2.54" size="1.778" layer="95"/>
 </segment>
+<segment>
+<wire x1="353.06" y1="-27.94" x2="353.06" y2="-15.24" width="0.1524" layer="91"/>
+<pinref part="C32" gate="G$1" pin="1"/>
+<junction x="353.06" y="-15.24"/>
+<label x="353.06" y="-17.78" size="1.778" layer="95"/>
+<junction x="353.06" y="-27.94"/>
+</segment>
 </net>
 <net name="VSS" class="2">
@@
 <junction x="398.78" y="7.62"/>
 </segment>
+<segment>
+<pinref part="C26" gate="G$1" pin="2"/>
+<wire x1="279.4" y1="-35.56" x2="292.1" y2="-35.56" width="0.1524" layer="91"/>
+<junction x="325.12" y="-35.56"/>
+<wire x1="292.1" y1="-35.56" x2="304.8" y2="-35.56" width="0.1524" layer="91"/>
+<wire x1="304.8" y1="-35.56" x2="320.04" y2="-35.56" width="0.1524" layer="91"/>
+<wire x1="320.04" y1="-35.56" x2="325.12" y2="-35.56" width="0.1524" layer="91"/>
+<wire x1="325.12" y1="-35.56" x2="332.74" y2="-35.56" width="0.1524" layer="91"/>
+<pinref part="VSS47" gate="G$1" pin="VSS"/>
+<pinref part="C27" gate="G$1" pin="2"/>
+<junction x="292.1" y="-35.56"/>
+<pinref part="C28" gate="G$1" pin="2"/>
+<junction x="304.8" y="-35.56"/>
+<pinref part="C29" gate="G$1" pin="2"/>
+<junction x="320.04" y="-35.56"/>
+<pinref part="C30" gate="G$1" pin="2"/>
+<wire x1="332.74" y1="-35.56" x2="342.9" y2="-35.56" width="0.1524" layer="91"/>
+<junction x="332.74" y="-35.56"/>
+<pinref part="C31" gate="G$1" pin="2"/>
+<wire x1="342.9" y1="-35.56" x2="353.06" y2="-35.56" width="0.1524" layer="91"/>
+<junction x="342.9" y="-35.56"/>
+<pinref part="C32" gate="G$1" pin="2"/>
+<junction x="279.4" y="-35.56"/>
+<junction x="353.06" y="-35.56"/>
+</segment>
 </net>
 <net name="AVDD" class="2">
@@
 <junction x="254" y="7.62"/>
 </segment>
+<segment>
+<pinref part="C28" gate="G$1" pin="1"/>
+<wire x1="304.8" y1="-27.94" x2="304.8" y2="-30.48" width="0.1524" layer="91"/>
+<wire x1="304.8" y1="-15.24" x2="304.8" y2="-27.94" width="0.1524" layer="91"/>
+<junction x="304.8" y="-15.24"/>
+<label x="304.8" y="-17.78" size="1.778" layer="95"/>
+<junction x="304.8" y="-27.94"/>
+</segment>
 </net>
 <net name="SCK2" class="0">
@@
 <label x="246.38" y="12.7" size="1.778" layer="95"/>
 </segment>
+<segment>
+<wire x1="332.74" y1="-27.94" x2="332.74" y2="-15.24" width="0.1524" layer="91"/>
+<pinref part="C30" gate="G$1" pin="1"/>
+<junction x="332.74" y="-15.24"/>
+<label x="332.74" y="-17.78" size="1.778" layer="95"/>
+<junction x="332.74" y="-27.94"/>
+</segment>
 </net>
 <net name="SDI2" class="0">
@@
 <junction x="254" y="5.08"/>
 <label x="246.38" y="5.08" size="1.778" layer="95"/>
+</segment>
+<segment>
+<wire x1="292.1" y1="-27.94" x2="292.1" y2="-15.24" width="0.1524" layer="91"/>
+<pinref part="C27" gate="G$1" pin="1"/>
+<junction x="292.1" y="-15.24"/>
+<label x="292.1" y="-17.78" size="1.778" layer="95"/>
+<junction x="292.1" y="-27.94"/>
 </segment>
 </net>
@@
 <junction x="254" y="15.24"/>
 <label x="246.38" y="15.24" size="1.778" layer="95"/>
+</segment>
+<segment>
+<wire x1="342.9" y1="-27.94" x2="342.9" y2="-15.24" width="0.1524" layer="91"/>
+<pinref part="C31" gate="G$1" pin="1"/>
+<junction x="342.9" y="-15.24"/>
+<label x="342.9" y="-17.78" size="1.778" layer="95"/>
+<junction x="342.9" y="-27.94"/>
 </segment>
 </net>
@@
 </segment>
 <segment>
-<wire x1="238.76" y1="10.16" x2="266.7" y2="10.16" width="0.1524" layer="91"/>
+<wire x1="254" y1="10.16" x2="266.7" y2="10.16" width="0.1524" layer="91"/>
 <pinref part="IC3" gate="G$1" pin="PTA_BT_PRIO_/_RPK6"/>
 <junction x="266.7" y="10.16"/>
-<junction x="238.76" y="10.16"/>
+<junction x="254" y="10.16"/>
 <label x="236.22" y="10.16" size="1.778" layer="95"/>
+</segment>
+<segment>
+<wire x1="320.04" y1="-27.94" x2="320.04" y2="-15.24" width="0.1524" layer="91"/>
+<pinref part="C29" gate="G$1" pin="1"/>
+<junction x="320.04" y="-15.24"/>
+<label x="320.04" y="-17.78" size="1.778" layer="95"/>
+<junction x="320.04" y="-27.94"/>
 </segment>
 </net>
@@
 </segment>
 <segment>
-<wire x1="266.7" y1="2.54" x2="241.3" y2="2.54" width="0.1524" layer="91"/>
+<wire x1="266.7" y1="2.54" x2="254" y2="2.54" width="0.1524" layer="91"/>
 <pinref part="IC3" gate="G$1" pin="PTA_BT_ACTIVE_/_RPK7"/>
 <junction x="266.7" y="2.54"/>
-<junction x="241.3" y="2.54"/>
+<junction x="254" y="2.54"/>
 <label x="236.22" y="2.54" size="1.778" layer="95"/>
+</segment>
+<segment>
+<wire x1="279.4" y1="-15.24" x2="279.4" y2="-27.94" width="0.1524" layer="91"/>
+<pinref part="C26" gate="G$1" pin="1"/>
+<junction x="279.4" y="-15.24"/>
+<label x="269.24" y="-17.78" size="1.778" layer="95"/>
+<junction x="279.4" y="-27.94"/>
 </segment>
 </net>
@@
 </segment>
 <segment>
-<wire x1="256.54" y1="27.94" x2="266.7" y2="27.94" width="0.1524" layer="91"/>
+<wire x1="254" y1="27.94" x2="266.7" y2="27.94" width="0.1524" layer="91"/>
 <pinref part="IC3" gate="G$1" pin="CVDT7_/_ERXERR_/_RPC9"/>
 <junction x="266.7" y="27.94"/>
-<junction x="256.54" y="27.94"/>
+<junction x="254" y="27.94"/>
 <label x="238.76" y="27.94" size="1.778" layer="95"/>
 </segment>
@@
 </segment>
 <segment>
-<wire x1="256.54" y1="38.1" x2="266.7" y2="38.1" width="0.1524" layer="91"/>
+<wire x1="254" y1="38.1" x2="266.7" y2="38.1" width="0.1524" layer="91"/>
 <pinref part="IC3" gate="G$1" pin="CVDT13_/_ETXD0_/_RPC15"/>
 <junction x="266.7" y="38.1"/>
-<junction x="256.54" y="38.1"/>
+<junction x="254" y="38.1"/>
 <label x="236.22" y="38.1" size="1.778" layer="95"/>
 </segment>
@@
 </segment>
 <segment>
-<wire x1="261.62" y1="55.88" x2="266.7" y2="55.88" width="0.1524" layer="91"/>
+<wire x1="256.54" y1="55.88" x2="266.7" y2="55.88" width="0.1524" layer="91"/>
 <pinref part="IC3" gate="G$1" pin="AN2_/_CVD2_/_CVDR2_/_CVDT5_/_USBID_/_RPB2"/>
 <junction x="266.7" y="55.88"/>
-<junction x="261.62" y="55.88"/>
+<junction x="256.54" y="55.88"/>
 <label x="243.84" y="55.88" size="1.778" layer="95"/>
 </segment>

Commit message: up
Parts:
- added JP4: (no value), pinhead:PINHD-1X1
Connections:
- net VSS: now also JP4.1
Changed lines of the file:
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@@
 <part name="C31" library="rcl" library_urn="urn:adsk.eagle:library:334" deviceset="C-US" device="C0402" package3d_urn="urn:adsk.eagle:package:23626/2" value="10pf"/>
 <part name="C32" library="rcl" library_urn="urn:adsk.eagle:library:334" deviceset="C-US" device="C0402" package3d_urn="urn:adsk.eagle:package:23626/2" value="10pf"/>
+<part name="VSS48" library="supply1" library_urn="urn:adsk.eagle:library:371" deviceset="VSS" device=""/>
+<part name="JP4" library="pinhead" library_urn="urn:adsk.eagle:library:325" deviceset="PINHD-1X1" device="" package3d_urn="urn:adsk.eagle:package:22485/2"/>
 </parts>
 <sheets>
@@
 <attribute name="NAME" x="354.076" y="-29.845" size="1.778" layer="95"/>
 <attribute name="VALUE" x="354.076" y="-34.671" size="1.778" layer="96"/>
+</instance>
+<instance part="VSS48" gate="G$1" x="68.58" y="-48.26" smashed="yes">
+<attribute name="VALUE" x="66.04" y="-53.34" size="1.778" layer="96" rot="R90"/>
+</instance>
+<instance part="JP4" gate="G$1" x="71.12" y="-45.72" smashed="yes">
+<attribute name="NAME" x="64.77" y="-42.545" size="1.778" layer="95"/>
+<attribute name="VALUE" x="64.77" y="-50.8" size="1.778" layer="96"/>
 </instance>
 </instances>
@@
 <junction x="353.06" y="-35.56"/>
 </segment>
+<segment>
+<pinref part="JP4" gate="G$1" pin="1"/>
+<pinref part="VSS48" gate="G$1" pin="VSS"/>
+</segment>
 </net>

Commit message: update for JCLPCB
Parts:
- JP4: value (none) -> VSS
Changed lines of the file:
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@@
 <part name="C32" library="rcl" library_urn="urn:adsk.eagle:library:334" deviceset="C-US" device="C0402" package3d_urn="urn:adsk.eagle:package:23626/2" value="10pf"/>
 <part name="VSS48" library="supply1" library_urn="urn:adsk.eagle:library:371" deviceset="VSS" device=""/>
-<part name="JP4" library="pinhead" library_urn="urn:adsk.eagle:library:325" deviceset="PINHD-1X1" device="" package3d_urn="urn:adsk.eagle:package:22485/2"/>
+<part name="JP4" library="pinhead" library_urn="urn:adsk.eagle:library:325" deviceset="PINHD-1X1" device="" package3d_urn="urn:adsk.eagle:package:22485/2" value="VSS"/>
+<part name="FRAME1" library="frames" library_urn="urn:adsk.eagle:library:229" deviceset="FRAME_C_L" device="" value="1.0"/>
 </parts>
 <sheets>
@@
 <attribute name="NAME" x="64.77" y="-42.545" size="1.778" layer="95"/>
 <attribute name="VALUE" x="64.77" y="-50.8" size="1.778" layer="96"/>
+</instance>
+<instance part="FRAME1" gate="G$1" x="-121.92" y="-124.46" smashed="yes"/>
+<instance part="FRAME1" gate="G$2" x="330.2" y="-124.46" smashed="yes">
+<attribute name="LAST_DATE_TIME" x="342.9" y="-123.19" size="2.54" layer="94"/>
+<attribute name="SHEET" x="416.56" y="-123.19" size="2.54" layer="94"/>
+<attribute name="DRAWING_NAME" x="347.98" y="-105.41" size="2.54" layer="94"/>
 </instance>
 </instances>
@@
 <junction x="-101.6" y="66.04"/>
 <junction x="-114.3" y="66.04"/>
-<label x="-121.92" y="66.04" size="1.778" layer="95"/>
+<label x="-111.76" y="68.58" size="1.778" layer="95" rot="R90"/>
 </segment>
 <segment>
@@
 <junction x="-101.6" y="63.5"/>
 <junction x="-114.3" y="63.5"/>
-<label x="-121.92" y="63.5" size="1.778" layer="95"/>
+<label x="-114.3" y="60.96" size="1.778" layer="95" rot="R270"/>
 </segment>
 <segment>
@@
 <junction x="398.78" y="63.5"/>
 <junction x="424.18" y="63.5"/>
-<label x="416.56" y="63.5" size="1.778" layer="95"/>
-</segment>
-</net>
+<label x="411.48" y="63.5" size="1.778" layer="95"/>
+</segment>
+</net>
